File: PCB/CG_Robot_Friend.kicad_pcb (KiCad board)
At the start: 2 copper layers, 62.2 x 85.7 mm, 26 parts, among them J1 PROTO, J10 PROTO, J11 PROTO, J12 PROTO, J2 PROTO, J3 PROTO, J4 PROTO, J5 PROTO, J6 PROTO, J7 PROTO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

Commit message: update to v03
Parts:
- added J13: PROTO, Adafruit:Pin_Header_Straight_1x03_Pitch2.54mm_no_silk, F.Cu at (129.5, 58.4)
- added J14: PROTO, Adafruit:Pin_Header_Straight_1x03_Pitch2.54mm_no_silk, F.Cu at (129.5, 55.9)
- added J15: PROTO, Adafruit:Pin_Header_Straight_1x03_Pitch2.54mm_no_silk, F.Cu at (129.5, 53.3)
- J10, J11, J12: footprint Adafruit:Pin_Header_Straight_1x18_Pitch2.54mm_nosilk -> Adafruit:Pin_Header_Straight_1x09_Pitch2.54mm_nosilk
Routing:
- net GND: vias 14 -> 15
Other:
- outline, holes or cut-outs redrawn
- board text added: "2019-11-11 v03"
- board text removed: "2019-11-08 v01"

Commit message: update mechanical PCB design
to open up a few of the hidden Crickit connectors
Parts:
- removed J13, J14, J15: PROTO, Adafruit:Pin_Header_Straight_1x03_Pitch2.54mm_no_silk
- J10, J11, J12: footprint Adafruit:Pin_Header_Straight_1x09_Pitch2.54mm_nosilk -> Adafruit:Pin_Header_Straight_1x08_Pitch2.54mm_no_silk
Other:
- outline, holes or cut-outs redrawn
- board text added: "2019-11-20 v03"
- board text added: "GND 3V3"
- board text removed: "2019-11-11 v03"
