File: PCB/CG_Robot_Friend.sch (KiCad schematic (older format))
At the start: 14 parts, among them J1 PROTO, J10 PROTO, J11 PROTO, J12 PROTO, J2 PROTO, J3 PROTO, J4 PROTO, J5 PROTO, J6 PROTO, J7 PROTO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

Commit message: update to v03
Parts:
- added J13, J14, J15: PROTO, Adafruit:Pin_Header_Straight_1x03_Pitch2.54mm_no_silk, symbol conn:CONN_01X03
- J10, J11, J12: footprint Adafruit:Pin_Header_Straight_1x18_Pitch2.54mm_nosilk -> Adafruit:Pin_Header_Straight_1x09_Pitch2.54mm_nosilk; symbol conn:CONN_01X18 -> conn:CONN_01X09
Other:
- note added: "Prototyping Area"

Commit message: update mechanical PCB design
to open up a few of the hidden Crickit connectors
Parts:
- removed J13, J14, J15: PROTO, Adafruit:Pin_Header_Straight_1x03_Pitch2.54mm_no_silk, symbol conn:CONN_01X03
- J10, J11, J12: footprint Adafruit:Pin_Header_Straight_1x09_Pitch2.54mm_nosilk -> Adafruit:Pin_Header_Straight_1x08_Pitch2.54mm_no_silk; symbol conn:CONN_01X09 -> conn:CONN_01X08
Changed lines of the file:
@@
 Sheet 1 1
 Title "Robot_Friend_FeatherWing"
-Date "2019-11-11"
+Date "2019-11-20"
 Rev "v03"
 Comp "Cedar Grove Studios"
@@
 	6350 1525 6750 1525
 $Comp
-L conn:CONN_01X09 J10
+L conn:CONN_01X08 J10
 U 1 1 5DCD5878
-P 7300 1925
-F 0 "J10" H 7450 2075 50  0000 C CNN
-F 1 "PROTO" H 7500 1975 50  0000 C CNN
-F 2 "Adafruit:Pin_Header_Straight_1x09_Pitch2.54mm_nosilk" H 7300 1925 50  0001 C CNN
-F 3 "" H 7300 1925 50  0001 C CNN
-	1    7300 1925
+P 7300 1875
+F 0 "J10" H 7450 2025 50  0000 C CNN
+F 1 "PROTO" H 7500 1925 50  0000 C CNN
+F 2 "Adafruit:Pin_Header_Straight_1x08_Pitch2.54mm_no_silk" H 7300 1875 50  0001 C CNN
+F 3 "" H 7300 1875 50  0001 C CNN
+	1    7300 1875
 	-1   0    0    -1
 $EndComp
@@
 	3175 5525 3575 5525
 $Comp
-L conn:CONN_01X09 J11
+L conn:CONN_01X08 J11
 U 1 1 5DC90487
-P 8025 1925
-F 0 "J11" H 8175 2075 50  0000 C CNN
-F 1 "PROTO" H 8225 1975 50  0000 C CNN
-F 2 "Adafruit:Pin_Header_Straight_1x09_Pitch2.54mm_nosilk" H 8025 1925 50  0001 C CNN
-F 3 "" H 8025 1925 50  0001 C CNN
-	1    8025 1925
+P 8025 1875
+F 0 "J11" H 8175 2025 50  0000 C CNN
+F 1 "PROTO" H 8225 1925 50  0000 C CNN
+F 2 "Adafruit:Pin_Header_Straight_1x08_Pitch2.54mm_no_silk" H 8025 1875 50  0001 C CNN
+F 3 "" H 8025 1875 50  0001 C CNN
+	1    8025 1875
 	-1   0    0    -1
 $EndComp
@@
 	8225 1525 8625 1525
 $Comp
-L conn:CONN_01X09 J12
+L conn:CONN_01X08 J12
 U 1 1 5DC90491
-P 8750 1925
-F 0 "J12" H 8900 2075 50  0000 C CNN
-F 1 "PROTO" H 8950 1975 50  0000 C CNN
-F 2 "Adafruit:Pin_Header_Straight_1x09_Pitch2.54mm_nosilk" H 8750 1925 50  0001 C CNN
-F 3 "" H 8750 1925 50  0001 C CNN
-	1    8750 1925
+P 8750 1875
+F 0 "J12" H 8900 2025 50  0000 C CNN
+F 1 "PROTO" H 8950 1925 50  0000 C CNN
+F 2 "Adafruit:Pin_Header_Straight_1x08_Pitch2.54mm_no_silk" H 8750 1875 50  0001 C CNN
+F 3 "" H 8750 1875 50  0001 C CNN
+	1    8750 1875
 	-1   0    0    -1
 $EndComp
@@
 Text Notes 5200 1250 0    50   ~ 0
 Prototyping Area
-$Comp
-L conn:CONN_01X03 J13
-U 1 1 5DCC6D06
-P 7300 3125
-F 0 "J13" H 7450 3275 50  0000 C CNN
-F 1 "PROTO" H 7500 3175 50  0000 C CNN
-F 2 "Adafruit:Pin_Header_Straight_1x03_Pitch2.54mm_no_silk" H 7300 3125 50  0001 C CNN
-F 3 "" H 7300 3125 50  0001 C CNN
-	1    7300 3125
-	-1   0    0    -1
-$EndComp
-$Comp
-L conn:CONN_01X03 J14
-U 1 1 5DCC6E29
-P 8025 3125
-F 0 "J14" H 8175 3275 50  0000 C CNN
-F 1 "PROTO" H 8225 3175 50  0000 C CNN
-F 2 "Adafruit:Pin_Header_Straight_1x03_Pitch2.54mm_no_silk" H 8025 3125 50  0001 C CNN
-F 3 "" H 8025 3125 50  0001 C CNN
-	1    8025 3125
-	-1   0    0    -1
-$EndComp
-$Comp
-L conn:CONN_01X03 J15
-U 1 1 5DCCDC6A
-P 8750 3125
-F 0 "J15" H 8900 3275 50  0000 C CNN
-F 1 "PROTO" H 8950 3175 50  0000 C CNN
-F 2 "Adafruit:Pin_Header_Straight_1x03_Pitch2.54mm_no_silk" H 8750 3125 50  0001 C CNN
-F 3 "" H 8750 3125 50  0001 C CNN
-	1    8750 3125
-	-1   0    0    -1
-$EndComp
 $EndSCHEMATC
